File: hardware_pcb/aries/aries.kicad_pcb (KiCad board)
At the start: 2 copper layers, 48 x 75 mm, 6 parts, among them J1 Conn_01x07_Socket (TFT Displa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, U1 XIAO_ESP32C3, U2 SCD40-D-R2

Commit message: changed to the mocking jay
Parts:
- moved G*** 3.00 mm to (124.0, 122.5)
